File: hardware/drone_lab_air/drone_lab_air.kicad_sch (KiCad schematic)
At the start: 0 parts

Commit message: Basic hierachical sheets
Other:
- added sheet Battery Manager (bms.kicad_sch)
- added sheet IHM (ihm.kicad_sch)
- added sheet IMU MPU6050 (imu_mpu6050.kicad_sch)
- added sheet IMU MPU9250 (imu_mpu9250.kicad_sch)
- added sheet MCU (mcu.kicad_sch)
- added sheet Motor Interface (motor_interface.kicad_sch)
- added sheet Power Supply (power_supply.kicad_sch)
