File: hardware/drone_lab_air/mcu.kicad_sch (KiCad schematic)
At the start: 0 parts

Commit message: Teensy library added
Parts:
- added U1: Teensy4.1, teensy.pretty-master:Teensy41, symbol teensy:Teensy4.1
Changed lines of the file:
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@@
 	(generator_version "9.0")
 	(paper "A4")
+	(symbol
+		(lib_id "teensy:Teensy4.1")
+		(at 139.7 113.03 0)
+		(unit 1)
+		(exclude_from_sim no)
+		(in_bom yes)
+		(on_board yes)
+		(dnp no)
+		(fields_autoplaced yes)
+		(property "Reference" "U1"
+			(at 139.7 46.99 0)
+			(effects
+				(font
+					(size 1.27 1.27)
+				)
+			)
+		)
+		(property "Value" "Teensy4.1"
+			(at 139.7 49.53 0)
+			(effects
+				(font
+					(size 1.27 1.27)
+				)
+			)
+		)
+		(property "Footprint" "teensy.pretty-master:Teensy41"
+			(at 129.54 102.87 0)
+			(effects
+				(font
+					(size 1.27 1.27)
+				)
+				(hide yes)
+			)
+		)
+		(property "Datasheet" ""
+			(at 129.54 102.87 0)
+			(effects
+				(font
+					(size 1.27 1.27)
+				)
+				(hide yes)
+			)
+		)
+		(property "Description" ""
+			(at 139.7 113.03 0)
+			(effects
+				(font
+					(size 1.27 1.27)
+				)
+				(hide yes)
+			)
+		)
+		(pin "36"
+		)
+		(pin "31"
+		)
+		(pin "22"
+		)
+		(pin "34"
+		)
+		(pin "55"
+		)
+		(pin "37"
+		)
+		(pin "40"
+		)
+		(pin "39"
+		)
+		(pin "59"
+		)
+		(pin "48"
+		)
+		(pin "21"
+		)
+		(pin "9"
+		)
+		(pin "7"
+		)
+		(pin "60"
+		)
+		(pin "65"
+		)
+		(pin "16"
+		)
+		(pin "19"
+		)
+		(pin "12"
+		)
+		(pin "17"
+		)
+		(pin "10"
+		)
+		(pin "5"
+		)
+		(pin "6"
+		)
+		(pin "4"
+		)
+		(pin "3"
+		)
+		(pin "8"
+		)
+		(pin "11"
+		)
+		(pin "63"
+		)
+		(pin "62"
+		)
+		(pin "61"
+		)
+		(pin "64"
+		)
+		(pin "2"
+		)
+		(pin "52"
+		)
+		(pin "38"
+		)
+		(pin "24"
+		)
+		(pin "27"
+		)
+		(pin "30"
+		)
+		(pin "44"
+		)
+		(pin "56"
+		)
+		(pin "1"
+		)
+		(pin "41"
+		)
+		(pin "32"
+		)
+		(pin "53"
+		)
+		(pin "54"
+		)
+		(pin "13"
+		)
+		(pin "47"
+		)
+		(pin "67"
+		)
+		(pin "18"
+		)
+		(pin "66"
+		)
+		(pin "51"
+		)
+		(pin "45"
+		)
+		(pin "26"
+		)
+		(pin "14"
+		)
+		(pin "15"
+		)
+		(pin "57"
+		)
+		(pin "29"
+		)
+		(pin "58"
+		)
+		(pin "25"
+		)
+		(pin "33"
+		)
+		(pin "23"
+		)
+		(pin "42"
+		)
+		(pin "43"
+		)
+		(pin "28"
+		)
+		(pin "46"
+		)
+		(pin "35"
+		)
+		(pin "49"
+		)
+		(pin "50"
+		)
+		(pin "20"
+		)
+		(instances
+			(project ""
+				(path "/ceb765fc-47c7-4cc0-8145-c04bbb330765/56ac78c1-8542-4c16-adfd-3ec3935b947c"
+					(reference "U1")
+					(unit 1)
+				)
+			)
+		)
+	)
 )
